File: WifiDriverREV2.brd (EAGLE design)
At the start: 99 x 70.8 mm, 7 parts, among them U1 ESP32-DEVKITC-32U, U2 ESP32-DEVKITC-32U, U3 DS18B20

Commit message: rev 2 schematic
Parts:
- added J1: (no value), SparkFun-Connectors:SCREWTERMINAL-3.5MM-2_LOCK
- moved U3 24.3 mm to (40.8, 11.7)
- moved R1 19.9 mm to (41.1, 6.35)
Connections:
- net 5V: now also J1.1
- net GND: now also J1.2
Routing:
- net DQ: track 149.3 -> 66.2 mm
- net 5V: track 98.5 -> 127.0 mm
